Commit message: change calibration and sensor xacro

File: logiee_sensor_kit_description/urdf/sensors.xacro (robot description, xacro)
@@ -1,20 +1,11 @@
 <?xml version="1.0"?>
 <robot name="vehicle" xmlns:xacro="http://ros.org/wiki/xacro">
-  <xacro:arg name="config_dir" default="$(find logiee_sensor_kit_description)/config"/>
-  <xacro:property name="calibration" value="${xacro.load_yaml('$(arg config_dir)/sensors_calibration.yaml')}"/>
-  <!-- sensor kit -->
-  <xacro:include filename="sensor_kit.xacro"/>
-  <xacro:sensor_kit_macro
-    parent="base_link"
-    x="${calibration['base_link']['sensor_kit_base_link']['x']}"
-    y="${calibration['base_link']['sensor_kit_base_link']['y']}"
-    z="${calibration['base_link']['sensor_kit_base_link']['z']}"
-    roll="${calibration['base_link']['sensor_kit_base_link']['roll']}"
-    pitch="${calibration['base_link']['sensor_kit_base_link']['pitch']}"
-    yaw="${calibration['base_link']['sensor_kit_base_link']['yaw']}"
-  />
-  <!-- embedded sensors -->
+  <xacro:arg name="config_dir" default="$(find sample_diff_drive_sensor_kit_description)/config"/>
+  <xacro:property name="calibration" value="${load_yaml('$(arg config_dir)/sensors_calibration.yaml')}"/>
+  <!-- rm if vehicle urdf spawn -->
+  <!--link name="base_link" /-->
+  <!-- lidar -->
   <xacro:include filename="$(find velodyne_description)/urdf/VLP-16.urdf.xacro"/>
-  <xacro:VLP-16 parent="base_link" name="velodyne_rear" topic="velodyne_rear/velodyne_points" hz="10" samples="220" gpu="false">
+  <xacro:VLP-16 parent="base_link" name="velodyne_rear" topic="/points_raw" hz="10" samples="220" gpu="false">
     <origin
       xyz="${calibration['base_link']['velodyne_rear_base_link']['x']}
@@ -26,3 +17,26 @@
     />
   </xacro:VLP-16>
+  <xacro:VLP-16 parent="base_link" name="velodyne_top" topic="/points_raw" hz="10" samples="220" gpu="false">
+    <origin
+      xyz="${calibration['base_link']['velodyne_top_base_link']['x']}
+           ${calibration['base_link']['velodyne_top_base_link']['y']}
+           ${calibration['base_link']['velodyne_top_base_link']['z']}"
+      rpy="${calibration['base_link']['velodyne_top_base_link']['roll']}
+           ${calibration['base_link']['velodyne_top_base_link']['pitch']}
+           ${calibration['base_link']['velodyne_top_base_link']['yaw']}"
+    />
+  </xacro:VLP-16>
+  <link name="imu_link"/>
+  <joint name="base_link_to_imu" type="fixed">
+    <parent link="base_link"/>
+    <child link="imu_link"/>
+    <origin
+        xyz="${calibration['base_link']['imu_link']['x']}
+            ${calibration['base_link']['imu_link']['y']}
+            ${calibration['base_link']['imu_link']['z']}"
+        rpy="${calibration['base_link']['imu_link']['roll']}
+            ${calibration['base_link']['imu_link']['pitch']}
+            ${calibration['base_link']['imu_link']['yaw']}"
+    />
+  </joint>
 </robot>

Commit message: update sensor_param

File: logiee_sensor_kit_description/urdf/sensors.xacro (robot description, xacro)
@@ -2,19 +2,10 @@
 <robot name="vehicle" xmlns:xacro="http://ros.org/wiki/xacro">
   <xacro:arg name="config_dir" default="$(find logiee_sensor_kit_description)/config"/>
-  <xacro:property name="calibration" value="${xacro.load_yaml('$(arg config_dir)/sensors_calibration.yaml')}"/>
-  <!-- sensor kit -->
-  <xacro:include filename="sensor_kit.xacro"/>
-  <xacro:sensor_kit_macro
-    parent="base_link"
-    x="${calibration['base_link']['sensor_kit_base_link']['x']}"
-    y="${calibration['base_link']['sensor_kit_base_link']['y']}"
-    z="${calibration['base_link']['sensor_kit_base_link']['z']}"
-    roll="${calibration['base_link']['sensor_kit_base_link']['roll']}"
-    pitch="${calibration['base_link']['sensor_kit_base_link']['pitch']}"
-    yaw="${calibration['base_link']['sensor_kit_base_link']['yaw']}"
-  />
-  <!-- embedded sensors -->
+  <xacro:property name="calibration" value="${load_yaml('$(arg config_dir)/sensors_calibration.yaml')}"/>
+  <!-- rm if vehicle urdf spawn -->
+  <!--link name="base_link" /-->
+  <!-- lidar -->
   <xacro:include filename="$(find velodyne_description)/urdf/VLP-16.urdf.xacro"/>
-  <xacro:VLP-16 parent="base_link" name="velodyne_rear" topic="velodyne_rear/velodyne_points" hz="10" samples="220" gpu="false">
+  <xacro:VLP-16 parent="base_link" name="velodyne_rear" topic="/points_raw" hz="10" samples="220" gpu="false">
     <origin
       xyz="${calibration['base_link']['velodyne_rear_base_link']['x']}
@@ -26,3 +17,26 @@
     />
   </xacro:VLP-16>
+  <xacro:VLP-16 parent="base_link" name="velodyne_top" topic="/points_raw" hz="10" samples="220" gpu="false">
+    <origin
+      xyz="${calibration['base_link']['velodyne_top_base_link']['x']}
+           ${calibration['base_link']['velodyne_top_base_link']['y']}
+           ${calibration['base_link']['velodyne_top_base_link']['z']}"
+      rpy="${calibration['base_link']['velodyne_top_base_link']['roll']}
+           ${calibration['base_link']['velodyne_top_base_link']['pitch']}
+           ${calibration['base_link']['velodyne_top_base_link']['yaw']}"
+    />
+  </xacro:VLP-16>
+  <link name="imu_link"/>
+  <joint name="base_link_to_imu" type="fixed">
+    <parent link="base_link"/>
+    <child link="imu_link"/>
+    <origin
+        xyz="${calibration['base_link']['imu_link']['x']}
+            ${calibration['base_link']['imu_link']['y']}
+            ${calibration['base_link']['imu_link']['z']}"
+        rpy="${calibration['base_link']['imu_link']['roll']}
+            ${calibration['base_link']['imu_link']['pitch']}
+            ${calibration['base_link']['imu_link']['yaw']}"
+    />
+  </joint>
 </robot>
